Commit message: Imu verileri düzeltildi

File: vehicle_description/urdf/vehicle_core.urdf.xacro (robot description, xacro)
@@ -43,10 +43,10 @@
         <parent link="vehicle_body"/>
         <child link="imu2_link"/>
-        <origin xyz="0 0 ${(body_height / 2) + 0.01 + wheel_radius}"/>
+        <origin xyz="0 0 ${(body_height / 2) + 0.01 + wheel_radius}" rpy="0 0 0"/>
     </joint>
     <joint name="imu_joint_3" type="fixed">
         <parent link="vehicle_body"/>
         <child link="imu3_link"/>
-        <origin xyz="${-0.05} 0 ${(body_height / 2) + 0.01 + wheel_radius}"/>
+        <origin xyz="${-0.05} 0 ${(body_height / 2) + 0.01 + wheel_radius}" rpy="0 0 0"/>
     </joint>
 </robot>

File: vehicle_description/urdf/vehicle_gazebo.xacro (robot description, xacro)
@@ -32,7 +32,8 @@
             <parameters>$(find vehicle_description)/config/vehicle_controller.yaml</parameters>
         </plugin>
-        <plugin filename="ignition-gazebo-imu-system" name="ignition::gazebo::systems::Imu"/>
+        <plugin filename="ignition-gazebo-imu-system" name="ignition::gazebo::systems::Imu">
+        </plugin>
         <plugin filename="ignition-gazebo-sensors-system" name="ignition::gazebo::systems::Sensors">
-            <renger_engine>ogre2</renger_engine>
+            <render_engine>ogre2</render_engine>
         </plugin>
     </gazebo>

File: vehicle_description/urdf/vehicle_gazebo_controls.xacro (robot description, xacro)
@@ -2,5 +2,5 @@
 <robot name="vehicle" xmlns:xacro="http://ros.org/wiki/xacro">
     <!-- Donanım ile etkileşime geçen kısmı ayarladığımız nokta !! -->
-    <ros2_control name="VehicleSystem" type="system" >
+    <ros2_control name="RobotSystem" type="system" >
         <hardware>
             <plugin>ign_ros2_control/IgnitionSystem</plugin>

File: vehicle_description/urdf/vehicle_materials.xacro (robot description, xacro)
@@ -102,14 +102,14 @@
                 <origin xyz="0 0 0"/>
                 <geometry>
-                    <box size="0.05 0.05 0.02"/>
+                    <box size="0.05 0.05 0.01"/>
                 </geometry>
             </collision>
             <inertial>
                 <origin xyz="0 0 0" rpy="0 0 0" />
-                <mass value="0.1" />
-                <inertia ixx="${(1 / 12) * 0.4 * (0.05 * 0.05 + 0.02 * 0.02)}"
-                         iyy="${(1 / 12) * 0.4 * (0.05 * 0.05 + 0.02 * 0.02)}"
-                         izz="${(1 / 12) * 0.4 * (0.05 * 0.05 + 0.05 * 0.05)}"
-                         ixy="0" ixz="0" iyz="0" iyx="0" izx="0" izy="0"
+                <mass value="0.05" />
+                <inertia ixx="${(1 / 12) * 0.05 * (0.05 * 0.05 + 0.01 * 0.01)}"
+                         iyy="${(1 / 12) * 0.05 * (0.05 * 0.05 + 0.01 * 0.01)}"
+                         izz="${(1 / 12) * 0.05 * (0.05 * 0.05 + 0.05 * 0.05)}"
+                         ixy="0" ixz="0" iyz="0"
                 />
             </inertial>

Commit message: Optimization, imu_logger

File: vehicle_description/urdf/vehicle_core.urdf.xacro (robot description, xacro)
@@ -20,4 +20,5 @@
         <origin xyz="${-(body_width / 4)} ${((body_depth / 2) + (wheel_length / 2))} 0" rpy="-${pi/2} 0 0"/>
         <axis xyz="0 0 1"/>
+        <!-- <dynamics damping="0.2" /> -->
     </joint>
     <joint name="rear_left_wheel_joint" type="continuous">
@@ -26,4 +27,5 @@
         <origin xyz="${-(body_width / 4)} ${-((body_depth / 2) + (wheel_length / 2))} 0" rpy="-${pi/2} 0 0"/>
         <axis xyz="0 0 1"/>
+        <!-- <dynamics damping="0.2" /> -->
     </joint>
     <joint name="front_caster_wheel_joint" type="fixed">

File: vehicle_description/urdf/vehicle_gazebo.xacro (robot description, xacro)
@@ -28,4 +28,5 @@
         <fdirl>1 0 0</fdirl>
     </gazebo>
+    <!-- -->
     <gazebo>
         <plugin filename="ign_ros2_control-system" name="ign_ros2_control::IgnitionROS2ControlPlugin">

File: vehicle_description/urdf/vehicle_gazebo_controls.xacro (robot description, xacro)
@@ -2,12 +2,16 @@
 <robot name="vehicle" xmlns:xacro="http://ros.org/wiki/xacro">
     <!-- Donanım ile etkileşime geçen kısmı ayarladığımız nokta !! -->
-    <ros2_control name="RobotSystem" type="system" >
+    <ros2_control name="DiffSystem" type="system" >
+        <!-- use mock hardware gerçek bir robota yükleme yaparken kullanılır! -->
         <hardware>
             <plugin>ign_ros2_control/IgnitionSystem</plugin>
+            <!-- Donanımın default başlatma-durdurma süresini belirleriz -->
+            <param name="example_param_hw_start_duration_sec">0</param>
+            <param name="example_param_hw_stop_duration_sec">3.0</param>
         </hardware>
         <joint name="rear_right_wheel_joint">
             <command_interface name="velocity">
-                <param name="min">-2</param>
-                <param name="max">2</param>
+                <param name="min">-1</param>
+                <param name="max">1</param>
             </command_interface>
             <state_interface name="position" />
@@ -16,6 +20,6 @@
         <joint name="rear_left_wheel_joint">
             <command_interface name="velocity">
-                <param name="min">-2</param>
-                <param name="max">2</param>
+                <param name="min">-1</param>
+                <param name="max">1</param>
             </command_interface>
             <state_interface name="position" />

Commit message: Dosya düzeni değiştirildi!

File: vehicle_description/urdf/vehicle_core.urdf.xacro (robot description, xacro)
@@ -1,54 +1,16 @@
 <?xml version="1.0"?>
-<robot name="vehicle" xmlns:xacro="http://ros.org/wiki/xacro">
+<robot name="vehicle" xmlns:xacro="http://www.ros.org/wiki/xacro">
     <xacro:arg name="is_ignition" default="true" />
-    <xacro:include filename="$(find vehicle_description)/urdf/vehicle_materials.xacro" />
-    <xacro:include filename="$(find vehicle_description)/urdf/vehicle_gazebo.xacro" />
-    <xacro:include filename="$(find vehicle_description)/urdf/vehicle_gazebo_controls.xacro"/>
-    <link name="base_footprint" />
+    <xacro:include filename="$(find vehicle_description)/urdf/includes.xacro" />
     <xacro:vehicle_body />
-    <joint name="base_joint" type="fixed">
-        <parent link="base_footprint"/>
-        <child link="vehicle_body"/>
-        <origin xyz="0 0 ${body_height / 2}"/>
-    </joint>
-    <xacro:wheel prefix="rear_right" />
-    <xacro:wheel prefix="rear_left" />
-    <xacro:caster_wheel prefix="front" />
-    <joint name="rear_right_wheel_joint" type="continuous">
-        <parent link="vehicle_body"/>
-        <child link="rear_right_wheel"/>
-        <origin xyz="${-(body_width / 4)} ${((body_depth / 2) + (wheel_length / 2))} 0" rpy="-${pi/2} 0 0"/>
-        <axis xyz="0 0 1"/>
-        <!-- <dynamics damping="0.2" /> -->
-    </joint>
-    <joint name="rear_left_wheel_joint" type="continuous">
-        <parent link="vehicle_body"/>
-        <child link="rear_left_wheel"/>
-        <origin xyz="${-(body_width / 4)} ${-((body_depth / 2) + (wheel_length / 2))} 0" rpy="-${pi/2} 0 0"/>
-        <axis xyz="0 0 1"/>
-        <!-- <dynamics damping="0.2" /> -->
-    </joint>
-    <joint name="front_caster_wheel_joint" type="fixed">
-        <parent link="vehicle_body"/>
-        <child  link="front_caster_wheel"/>
-        <origin xyz="${body_width / 4} 0 0"/>
-    </joint>
-    <xacro:imu prefix="imu1" />
-    <xacro:imu prefix="imu2" />
-    <xacro:imu prefix="imu3" />
-    <joint name="imu_joint_1" type="fixed">
-        <parent link="vehicle_body"/>
-        <child link="imu1_link"/>
-        <origin xyz="${0.05} 0 ${(body_height / 2) + 0.01 + wheel_radius}" rpy="0 0 0"/>
-    </joint>
-    <joint name="imu_joint_2" type="fixed">
-        <parent link="vehicle_body"/>
-        <child link="imu2_link"/>
-        <origin xyz="0 0 ${(body_height / 2) + 0.01 + wheel_radius}" rpy="0 0 0"/>
-    </joint>
-    <joint name="imu_joint_3" type="fixed">
-        <parent link="vehicle_body"/>
-        <child link="imu3_link"/>
-        <origin xyz="${-0.05} 0 ${(body_height / 2) + 0.01 + wheel_radius}" rpy="0 0 0"/>
-    </joint>
+    <xacro:vehicle_wheels parent="vehicle_body"/>
+    <xacro:imu_sensor name="imu1" topic_ns="imu1" parent="vehicle_body">
+        <origin xyz="0.05 0 ${(body_height / 2) + wheel_radius}" rpy="-${pi/2} 0 0"/>
+    </xacro:imu_sensor>
+    <xacro:imu_sensor name="imu2" topic_ns="imu2" parent="vehicle_body">
+        <origin xyz="0 0 ${(body_height / 2) + wheel_radius}" rpy="-${pi/2} 0 0"></origin>
+    </xacro:imu_sensor>
+    <xacro:imu_sensor name="imu3" topic_ns="imu3" parent="vehicle_body">
+        <origin xyz="-0.05 0 ${(body_height / 2) + wheel_radius}" rpy="-${pi/2} 0 0"></origin>
+    </xacro:imu_sensor>
 </robot>
