Commit message: Imu logger optimize edildi ve imu_sensor.xacro dosyasındaki hatalar düzeltildi

File: vehicle_description/urdf/includes.xacro (robot description, xacro)
@@ -9,5 +9,5 @@
     <xacro:include filename="$(find vehicle_description)/urdf/includes/components/wheels/vehicle_wheels.xacro" />
     <!-- IMU -->
-    <xacro:include filename="$(find vehicle_description)/urdf/includes/components/sensors/bno055.xacro"/>
+    <xacro:include filename="$(find vehicle_description)/urdf/includes/components/sensors/imu_sensor.xacro" />
     <!-- Gazebo configurations-->
     <xacro:include filename="$(find vehicle_description)/urdf/includes/gazebo/gazebo_system.xacro" />

File: vehicle_description/urdf/includes/components/sensors/bno055.xacro (robot description, xacro)
@@ -3,9 +3,4 @@
     <!-- Gazebo IMU plugin -->
     <xacro:include filename="$(find vehicle_description)/urdf/includes/components/sensors/imu_gazebo.xacro" />
-    <!-- VN100 CONSTANST https://www.vectornav.com/docs/default-source/product-brief/vn-100-product-brief.pdf?sfvrsn=a2a5ae5f_2 -->
-    <xacro:property name="vn100_depth" value="0.022" />
-    <xacro:property name="vn100_width" value="0.024" />
-    <xacro:property name="vn100_height" value="0.003"/>
-    <xacro:property name="vn100_mass" value="0.0035"/>
     <!-- Kaynak: https://www.mouser.com.tr/ProductDetail/Bosch-Sensortec/BNO055?qs=QhAb4EtQfbV8Z2YmISucWw%3D%3D&srsltid=AfmBOoqaJM1CKMs2fuZsgKlemHZyKtVKounwW_lcwwsTkwHkVq9O6MgB -->
     <xacro:property name="bno_depth" value="0.0052" />
@@ -13,5 +8,5 @@
     <xacro:property name="bno_height" value="0.00113"/>
     <xacro:property name="bno_mass" value="0.00015"/>
-    <xacro:macro name="imu_sensor" params="name topic_ns:=imu parent *origin">
+    <xacro:macro name="bno_055" params="name topic_ns:=imu parent *origin">
         <joint name="${name}_joint" type="fixed">
             <parent link="${parent}"/>
@@ -37,29 +32,3 @@
         <xacro:imu_gazebo_bno055  imu_name="${name}" topic_ns="${topic_ns}" />
     </xacro:macro>
-    <!--
-    <xacro:macro name="imu_sensor" params="name topic_ns:=imu parent *origin">
-        <joint name="${name}_joint" type="fixed">
-            <parent link="${parent}"/>
-            <child link="${name}_link"/>
-            <xacro:insert_block name="origin" />
-        </joint>
-        <link name="${name}_link">
-            <visual>
-                <origin xyz="0 0 0"/>
-                <geometry>
-                    <box size="${vn100_width} ${vn100_depth} ${vn100_height}"/>
-                </geometry>
-                <material name="silver" />
-            </visual>
-            <collision>
-                <origin xyz="0 0 0"/>
-                <geometry>
-                    <box size="${vn100_width} ${vn100_depth} ${vn100_height}"/>
-                </geometry>
-            </collision>
-            <xacro:solid_cuboid_inertia mass="${vn100_mass}" x="${vn100_width}" y="${vn100_depth}" z="${bno_height}" />
-        </link>
-        <xacro:imu_gazebo_VN100 imu_name="${name}" topic_ns="${topic_ns}" />
-    </xacro:macro>
-    -->
 </robot>

File: vehicle_description/urdf/includes/components/sensors/imu_gazebo.xacro (robot description, xacro)
@@ -2,4 +2,5 @@
 <robot name="vehicle" xmlns:xacro="http://www.ros.org/wiki/xacro">
     <!-- IMU Plugin -->
+    <!-- Şimdilik kullanımdan kaldırılmıştır!! -->
     <xacro:macro name="imu_gazebo_bno055" params="imu_name topic_ns" >
         <gazebo reference="${name}_link">
@@ -16,7 +17,7 @@
                             <noise type="gaussian">
                                 <mean>0.0</mean>
-                                <stddev>0.00523598775</stddev>  <!-- Noise Density -->
+                                <stddev>0.001745329251</stddev>  <!-- Noise Density, radyan cinsinden! (sensörün tipik davranışı modellenmiştir) -->
                                 <bias_mean>0.0</bias_mean>
-                                <bias_stddev>0.05235987755</bias_stddev> <!-- Bias instability -->
+                                <bias_stddev>0.01745329251</bias_stddev> <!-- Bias instability, radyan cinsinden! (sensörün tipik davranışı modellenmiştir) -->
                             </noise>
                         </x>
@@ -24,7 +25,7 @@
                             <noise type="gaussian">
                                 <mean>0.0</mean>
-                                <stddev>0.00523598775</stddev>
+                                <stddev>0.001745329251</stddev>
                                 <bias_mean>0.0</bias_mean>
-                                <bias_stddev>0.0005235987755</bias_stddev>
+                                <bias_stddev>0.01745329251</bias_stddev>
                             </noise>
                         </y>
@@ -32,7 +33,7 @@
                             <noise type="gaussian">
                                 <mean>0.0</mean>
-                                <stddev>0.00523598775</stddev>
+                                <stddev>0.001745329251</stddev>
                                 <bias_mean>0.0</bias_mean>
-                                <bias_stddev>0.05235987755</bias_stddev>
+                                <bias_stddev>0.01745329251</bias_stddev>
                             </noise>
                         </z>
@@ -41,8 +42,8 @@
                         <x>
                             <noise type="gaussian">
-                                <mean>0.0</mean>
-                                <stddev>1.8639e-5</stddev>
+                                <mean>0.0</mean>    <!-- 100 ODR(Output Data Rate) için 32hz bandwith-->
+                                <stddev>8.32e-3</stddev> <!-- Output Noise Density, m/s^2 cinsinde, sensorün tipik davranışı ele alınmıştır. -->
                                 <bias_mean>0.0</bias_mean>
-                                <bias_stddev>1.471e-3</bias_stddev>
+                                <bias_stddev>0.4903</bias_stddev>
                             </noise>
                         </x>
@@ -82,7 +83,7 @@
                             <noise type="gaussian">
                                 <mean>0.0</mean>
-                                <stddev>0.000740</stddev>
+                                <stddev>9.94e-4</stddev>
                                 <bias_mean>0.0</bias_mean>
-                                <bias_stddev>0.008727</bias_stddev>
+                                <bias_stddev>4.848e-6</bias_stddev> <!-- radyan cinsinden -->
                             </noise>
                         </x>
@@ -90,7 +91,7 @@
                             <noise type="gaussian">
                                 <mean>0.0</mean>
-                                <stddev>0.000740</stddev>
+                                <stddev>9.94e-4</stddev>
                                 <bias_mean>0.0</bias_mean>
-                                <bias_stddev>0.008727</bias_stddev>
+                                <bias_stddev>4.848e-6</bias_stddev>
                             </noise>
                         </y>
@@ -98,17 +99,17 @@
                             <noise type="gaussian">
                                 <mean>0.0</mean>
-                                <stddev>0.000740</stddev>
+                                <stddev>9.94e-4</stddev>
                                 <bias_mean>0.0</bias_mean>
-                                <bias_stddev>0.008727</bias_stddev>
+                                <bias_stddev>4.848e-6</bias_stddev>
                             </noise>
                         </z>
                     </angular_velocity>
-                    <linear_velocity>
+                    <linear_acceleration>
                         <x>
                             <noise type="gaussian">
                                 <mean>0.0</mean>
-                                <stddev>0.01665</stddev>
-                                <bias_mean></bias_mean>
-                                <bias_stddev>0.0002943</bias_stddev>
+                                <stddev>0.02082152953</stddev>
+                                <bias_mean>0.0</bias_mean>
+                                <bias_stddev>3.92e-4</bias_stddev> <!-- m/s^2 cinsinden. -->
                             </noise>
                         </x>
@@ -116,7 +117,7 @@
                             <noise type="gaussian">
                                 <mean>0.0</mean>
-                                <stddev>0.01665</stddev>
-                                <bias_mean></bias_mean>
-                                <bias_stddev>0.0002943</bias_stddev>
+                                <stddev>0.02082152953</stddev>
+                                <bias_mean>0.0</bias_mean>
+                                <bias_stddev>3.92e-4</bias_stddev>
                             </noise>
                         </y>
@@ -124,10 +125,10 @@
                             <noise type="gaussian">
                                 <mean>0.0</mean>
-                                <stddev>0.01665</stddev>
-                                <bias_mean></bias_mean>
-                                <bias_stddev>0.0002943</bias_stddev>
+                                <stddev>0.02082152953</stddev>
+                                <bias_mean>0.0</bias_mean>
+                                <bias_stddev>3.92e-4</bias_stddev>
                             </noise>
                         </z>
-                    </linear_velocity>
+                    </linear_acceleration>
                 </imu>
             </sensor>

File: vehicle_description/urdf/vehicle_core.urdf.xacro (robot description, xacro)
@@ -5,11 +5,11 @@
     <xacro:vehicle_body />
     <xacro:vehicle_wheels parent="vehicle_body"/>
-    <xacro:imu_sensor name="imu1" topic_ns="imu1" parent="vehicle_body">
+    <xacro:imu_sensor sensor_type="vn_100" name="imu1" topic_ns="imu1" parent="vehicle_body">
         <origin xyz="0 0 ${(body_height / 2) + wheel_radius}" rpy="0 0 0"/>
     </xacro:imu_sensor>
-    <xacro:imu_sensor name="imu2" topic_ns="imu2" parent="vehicle_body">
+    <xacro:imu_sensor sensor_type="vn_100" name="imu2" topic_ns="imu2" parent="vehicle_body">
         <origin xyz="0 0 ${(body_height / 2) + wheel_radius}" rpy="0 0 0"/>
     </xacro:imu_sensor>
-    <xacro:imu_sensor name="imu3" topic_ns="imu3" parent="vehicle_body">
+    <xacro:imu_sensor sensor_type="vn_100" name="imu3" topic_ns="imu3" parent="vehicle_body">
         <origin xyz="0 0 ${(body_height / 2) + wheel_radius}" rpy="0 0 0"/>
     </xacro:imu_sensor>

Commit message: Navsat, gps sensorü eklendi

File: vehicle_description/urdf/includes.xacro (robot description, xacro)
@@ -10,4 +10,6 @@
     <!-- IMU -->
     <xacro:include filename="$(find vehicle_description)/urdf/includes/components/sensors/imu_sensor.xacro" />
+    <!-- NAVSAT/GPS -->
+    <xacro:include filename="$(find vehicle_description)/urdf/includes/components/sensors/navsat_sensor.xacro" />
     <!-- Gazebo configurations-->
     <xacro:include filename="$(find vehicle_description)/urdf/includes/gazebo/gazebo_system.xacro" />

File: vehicle_description/urdf/includes/components/sensors/imu_gazebo.xacro (robot description, xacro)
@@ -70,11 +70,11 @@
     </xacro:macro>
     <xacro:macro name="imu_gazebo_VN100" params="imu_name topic_ns">
-        <gazebo reference="${name}_link">
+        <gazebo reference="${imu_name}_link">
             <!-- Based ON VN100 DATASHEET -->
             <!-- https://www.vectornav.com/docs/default-source/product-brief/vn-100-product-brief.pdf?sfvrsn=a2a5ae5f_2 -->
-            <sensor name="${name}" type="imu">
+            <sensor name="${imu_name}" type="imu">
                 <always_on>true</always_on>
                 <update_rate>200</update_rate>
-                <gz_fram_id>${name}_link</gz_fram_id>
+                <gz_fram_id>${imu_name}_link</gz_fram_id>
                 <topic>${topic_ns}</topic>
                 <imu>

File: vehicle_description/urdf/includes/gazebo/gazebo_system.xacro (robot description, xacro)
@@ -36,4 +36,5 @@
         </plugin>
         <plugin filename="ignition-gazebo-imu-system" name="ignition::gazebo::systems::Imu"></plugin>
+        <plugin filename="libignition-gazebo-navsat-system" name="ignition::gazebo::systems::NavSat"></plugin>
         <plugin filename="libignition-gazebo-sensors-system.so" name="ignition::gazebo::systems::Sensors">
             <render_engine>ogre2</render_engine>

File: vehicle_description/urdf/vehicle_core.urdf.xacro (robot description, xacro)
@@ -14,3 +14,6 @@
         <origin xyz="0 0 ${(body_height / 2) + wheel_radius}" rpy="0 0 0"/>
     </xacro:imu_sensor>
+    <xacro:navsat_sensor name="gps" topic_ns="navsat" parent="vehicle_body" >
+        <origin xyz="0.05 0 ${(body_height / 2) + wheel_radius}" rpy="0 0 0" />
+    </xacro:navsat_sensor>
 </robot>
