Commit message: BNO055 imu modellenmiştir

File: vehicle_description/urdf/includes/components/sensors/bno055.xacro (robot description, xacro)
@@ -2,10 +2,10 @@
 <robot name="vehicle" xmlns:xacro="http://www.ros.org/wiki/xacro">
     <!-- Gazebo IMU plugin -->
-    <!-- <xacro:include filename="$(find vehicle_description)/urdf/includes/components/sensors/imu_gazebo.xacro" /> -->
-    <!-- BNO055 Constants Kaynak: https://github.com/issaiass/jetbot_description/blob/f4be14f8498532d18ea53d2ff62d83b79504219f/urdf/includes/parts/sensors/imu/bno055.urdf.xacro -->
-    <xacro:property name="bno_depth" value="0.00254" />
-    <xacro:property name="bno_width" value="0.0254" />
-    <xacro:property name="bno_height" value="0.02032"/>
-    <xacro:property name="bno_mass" value="0.003"/>
+    <xacro:include filename="$(find vehicle_description)/urdf/includes/components/sensors/imu_gazebo.xacro" />
+    <!-- Kaynak: https://www.mouser.com.tr/ProductDetail/Bosch-Sensortec/BNO055?qs=QhAb4EtQfbV8Z2YmISucWw%3D%3D&srsltid=AfmBOoqaJM1CKMs2fuZsgKlemHZyKtVKounwW_lcwwsTkwHkVq9O6MgB -->
+    <xacro:property name="bno_depth" value="0.0052" />
+    <xacro:property name="bno_width" value="0.0038" />
+    <xacro:property name="bno_height" value="0.00113"/>
+    <xacro:property name="bno_mass" value="0.00015"/>
     <xacro:macro name="imu_sensor" params="name topic_ns:=imu parent *origin">
         <joint name="${name}_joint" type="fixed">
@@ -30,14 +30,5 @@
             <xacro:solid_cuboid_inertia mass="${bno_mass}" x="${bno_width}" y="${bno_depth}" z="${bno_height}" />
         </link>
-        <!-- <xacro:imu_gazebo  imu_name="${name}" topic_ns="${topic_ns}" /> -->
-        <gazebo reference="${name}_link">
-            <!-- Based on bno055 datasheet-->
-            <sensor name="${name}" type="imu">
-                <always_on>true</always_on>
-                <update_rate>100</update_rate>
-                <gz_frame_id>${name}_link</gz_frame_id>
-                <topic>${topic_ns}</topic>
-            </sensor>
-        </gazebo>
+        <xacro:imu_gazebo  imu_name="${name}" topic_ns="${topic_ns}" />
     </xacro:macro>
 </robot>

File: vehicle_description/urdf/includes/components/sensors/imu_gazebo.xacro (robot description, xacro)
@@ -3,11 +3,54 @@
     <!-- IMU Plugin -->
     <xacro:macro name="imu_gazebo" params="imu_name topic_ns" >
-        <gazebo reference="${imu_name}">
+        <gazebo reference="${name}_link">
             <!-- Based on bno055 datasheet-->
-            <sensor name="${name}">
+            <!-- https://www.bosch-sensortec.com/media/boschsensortec/downloads/datasheets/bst-bno055-ds000.pdf -->
+            <sensor name="${name}" type="imu">
                 <always_on>true</always_on>
-                <update_rate>75</update_rate>
-                <gz_frame_id>${imu_name}</gz_frame_id>
-                <topic>${imu_name}</topic>
+                <update_rate>100</update_rate>
+                <gz_frame_id>${name}_link</gz_frame_id>
+                <topic>${topic_ns}</topic>
+                <imu>
+                    <angular_velocity>
+                        <x>
+                        <noise type="gaussian">
+                            <mean>0.0</mean>
+                            <stddev>0.05236</stddev>
+                        </noise>
+                        </x>
+                        <y>
+                        <noise type="gaussian">
+                            <mean>0.0</mean>
+                            <stddev>0.05236</stddev>
+                        </noise>
+                        </y>
+                        <z>
+                        <noise type="gaussian">
+                            <mean>0.0</mean>
+                            <stddev>0.05236</stddev>
+                        </noise>
+                        </z>
+                    </angular_velocity>
+                    <linear_acceleration>
+                        <x>
+                        <noise type="gaussian">
+                            <mean>0.0</mean>
+                            <stddev>1.8639e-5</stddev>
+                        </noise>
+                        </x>
+                        <y>
+                        <noise type="gaussian">
+                            <mean>0.0</mean>
+                            <stddev>1.8639e-5</stddev>
+                        </noise>
+                        </y>
+                        <z>
+                        <noise type="gaussian">
+                            <mean>0.0</mean>
+                            <stddev>1.8639e-5</stddev>
+                        </noise>
+                        </z>
+                    </linear_acceleration>
+                </imu>
             </sensor>
         </gazebo>

File: vehicle_description/urdf/includes/gazebo/gazebo_system.xacro (robot description, xacro)
@@ -28,23 +28,21 @@
         <fdirl>1 0 0</fdirl>
     </gazebo>
-    <!-- -->
+    <!-- ?? -->
     <gazebo>
         <plugin filename="ign_ros2_control-system" name="ign_ros2_control::IgnitionROS2ControlPlugin">
+            <robot_param>robot_description</robot_param>
+            <robot_param_node>robot_state_publisher</robot_param_node>
             <parameters>$(find vehicle_description)/config/vehicle_controller.yaml</parameters>
         </plugin>
-        <plugin filename="ignition-gazebo-imu-system" name="ignition::gazebo::systems::Imu">
-        </plugin>
-        <plugin filename="ignition-gazebo-sensors-system" name="ignition::gazebo::systems::Sensors">
+        <plugin filename="ignition-gazebo-imu-system" name="ignition::gazebo::systems::Imu"></plugin>
+        <plugin filename="libignition-gazebo-sensors-system.so" name="ignition::gazebo::systems::Sensors">
             <render_engine>ogre2</render_engine>
         </plugin>
     </gazebo>
     <!-- Donanım ile etkileşime geçen kısmı ayarladığımız nokta !! -->
-    <ros2_control name="DiffSystem" type="system" >
+    <ros2_control name="IgnitionSystem" type="system" >
         <!-- use mock hardware gerçek bir robota yükleme yaparken kullanılır! -->
         <hardware>
             <plugin>ign_ros2_control/IgnitionSystem</plugin>
-            <!-- Donanımın default başlatma-durdurma süresini belirleriz -->
-            <param name="example_param_hw_start_duration_sec">0</param>
-            <param name="example_param_hw_stop_duration_sec">3.0</param>
         </hardware>
         <joint name="rear_right_wheel_joint">

File: vehicle_description/urdf/vehicle_core.urdf.xacro (robot description, xacro)
@@ -6,11 +6,11 @@
     <xacro:vehicle_wheels parent="vehicle_body"/>
     <xacro:imu_sensor name="imu1" topic_ns="imu1" parent="vehicle_body">
-        <origin xyz="0.05 0 ${(body_height / 2) + wheel_radius}" rpy="-${pi/2} 0 0"/>
+        <origin xyz="0.05 0 ${(body_height / 2) + wheel_radius}" rpy="0 0 0"/>
     </xacro:imu_sensor>
     <xacro:imu_sensor name="imu2" topic_ns="imu2" parent="vehicle_body">
-        <origin xyz="0 0 ${(body_height / 2) + wheel_radius}" rpy="-${pi/2} 0 0"></origin>
+        <origin xyz="0 0 ${(body_height / 2) + wheel_radius}" rpy="0 0 0"></origin>
     </xacro:imu_sensor>
     <xacro:imu_sensor name="imu3" topic_ns="imu3" parent="vehicle_body">
-        <origin xyz="-0.05 0 ${(body_height / 2) + wheel_radius}" rpy="-${pi/2} 0 0"></origin>
+        <origin xyz="-0.05 0 ${(body_height / 2) + wheel_radius}" rpy="0 0 0"></origin>
     </xacro:imu_sensor>
 </robot>

Commit message: Ekstra bir imu modeli eklendi vn100

File: vehicle_description/urdf/includes/components/sensors/bno055.xacro (robot description, xacro)
@@ -3,4 +3,9 @@
     <!-- Gazebo IMU plugin -->
     <xacro:include filename="$(find vehicle_description)/urdf/includes/components/sensors/imu_gazebo.xacro" />
+    <!-- VN100 CONSTANST https://www.vectornav.com/docs/default-source/product-brief/vn-100-product-brief.pdf?sfvrsn=a2a5ae5f_2 -->
+    <xacro:property name="vn100_depth" value="0.022" />
+    <xacro:property name="vn100_width" value="0.024" />
+    <xacro:property name="vn100_height" value="0.003"/>
+    <xacro:property name="vn100_mass" value="0.0035"/>
     <!-- Kaynak: https://www.mouser.com.tr/ProductDetail/Bosch-Sensortec/BNO055?qs=QhAb4EtQfbV8Z2YmISucWw%3D%3D&srsltid=AfmBOoqaJM1CKMs2fuZsgKlemHZyKtVKounwW_lcwwsTkwHkVq9O6MgB -->
     <xacro:property name="bno_depth" value="0.0052" />
@@ -30,5 +35,31 @@
             <xacro:solid_cuboid_inertia mass="${bno_mass}" x="${bno_width}" y="${bno_depth}" z="${bno_height}" />
         </link>
-        <xacro:imu_gazebo  imu_name="${name}" topic_ns="${topic_ns}" />
+        <xacro:imu_gazebo_bno055  imu_name="${name}" topic_ns="${topic_ns}" />
     </xacro:macro>
+    <!--
+    <xacro:macro name="imu_sensor" params="name topic_ns:=imu parent *origin">
+        <joint name="${name}_joint" type="fixed">
+            <parent link="${parent}"/>
+            <child link="${name}_link"/>
+            <xacro:insert_block name="origin" />
+        </joint>
+        <link name="${name}_link">
+            <visual>
+                <origin xyz="0 0 0"/>
+                <geometry>
+                    <box size="${vn100_width} ${vn100_depth} ${vn100_height}"/>
+                </geometry>
+                <material name="silver" />
+            </visual>
+            <collision>
+                <origin xyz="0 0 0"/>
+                <geometry>
+                    <box size="${vn100_width} ${vn100_depth} ${vn100_height}"/>
+                </geometry>
+            </collision>
+            <xacro:solid_cuboid_inertia mass="${vn100_mass}" x="${vn100_width}" y="${vn100_depth}" z="${bno_height}" />
+        </link>
+        <xacro:imu_gazebo_VN100 imu_name="${name}" topic_ns="${topic_ns}" />
+    </xacro:macro>
+    -->
 </robot>

File: vehicle_description/urdf/includes/components/sensors/imu_gazebo.xacro (robot description, xacro)
@@ -2,5 +2,5 @@
 <robot name="vehicle" xmlns:xacro="http://www.ros.org/wiki/xacro">
     <!-- IMU Plugin -->
-    <xacro:macro name="imu_gazebo" params="imu_name topic_ns" >
+    <xacro:macro name="imu_gazebo_bno055" params="imu_name topic_ns" >
         <gazebo reference="${name}_link">
             <!-- Based on bno055 datasheet-->
@@ -16,7 +16,7 @@
                             <noise type="gaussian">
                                 <mean>0.0</mean>
-                                <stddev>0.00523598775</stddev>
+                                <stddev>0.00523598775</stddev>  <!-- Noise Density -->
                                 <bias_mean>0.0</bias_mean>
-                                <bias_stddev>0.05235987755</bias_stddev>
+                                <bias_stddev>0.05235987755</bias_stddev> <!-- Bias instability -->
                             </noise>
                         </x>
@@ -68,3 +68,69 @@
         </gazebo>
     </xacro:macro>
+    <xacro:macro name="imu_gazebo_VN100" params="imu_name topic_ns">
+        <gazebo reference="${name}_link">
+            <!-- Based ON VN100 DATASHEET -->
+            <!-- https://www.vectornav.com/docs/default-source/product-brief/vn-100-product-brief.pdf?sfvrsn=a2a5ae5f_2 -->
+            <sensor name="${name}" type="imu">
+                <always_on>true</always_on>
+                <update_rate>200</update_rate>
+                <gz_fram_id>${name}_link</gz_fram_id>
+                <topic>${topic_ns}</topic>
+                <imu>
+                    <angular_velocity>
+                        <x>
+                            <noise type="gaussian">
+                                <mean>0.0</mean>
+                                <stddev>0.000740</stddev>
+                                <bias_mean>0.0</bias_mean>
+                                <bias_stddev>0.008727</bias_stddev>
+                            </noise>
+                        </x>
+                        <y>
+                            <noise type="gaussian">
+                                <mean>0.0</mean>
+                                <stddev>0.000740</stddev>
+                                <bias_mean>0.0</bias_mean>
+                                <bias_stddev>0.008727</bias_stddev>
+                            </noise>
+                        </y>
+                        <z>
+                            <noise type="gaussian">
+                                <mean>0.0</mean>
+                                <stddev>0.000740</stddev>
+                                <bias_mean>0.0</bias_mean>
+                                <bias_stddev>0.008727</bias_stddev>
+                            </noise>
+                        </z>
+                    </angular_velocity>
+                    <linear_velocity>
+                        <x>
+                            <noise type="gaussian">
+                                <mean>0.0</mean>
+                                <stddev>0.01665</stddev>
+                                <bias_mean></bias_mean>
+                                <bias_stddev>0.0002943</bias_stddev>
+                            </noise>
+                        </x>
+                        <y>
+                            <noise type="gaussian">
+                                <mean>0.0</mean>
+                                <stddev>0.01665</stddev>
+                                <bias_mean></bias_mean>
+                                <bias_stddev>0.0002943</bias_stddev>
+                            </noise>
+                        </y>
+                        <z>
+                            <noise type="gaussian">
+                                <mean>0.0</mean>
+                                <stddev>0.01665</stddev>
+                                <bias_mean></bias_mean>
+                                <bias_stddev>0.0002943</bias_stddev>
+                            </noise>
+                        </z>
+                    </linear_velocity>
+                </imu>
+            </sensor>
+        </gazebo>
+    </xacro:macro>
 </robot>
