Commit message: bno055 için bias değerleri eklendi

File: vehicle_description/urdf/includes/components/sensors/imu_gazebo.xacro (robot description, xacro)
@@ -14,28 +14,36 @@
                     <angular_velocity>
                         <x>
-                        <noise type="gaussian">
-                            <mean>0.0</mean>
-                            <stddev>0.05236</stddev>
-                        </noise>
+                            <noise type="gaussian">
+                                <mean>0.0</mean>
+                                <stddev>0.00523598775</stddev>
+                                <bias_mean>0.0</bias_mean>
+                                <bias_stddev>0.05235987755</bias_stddev>
+                            </noise>
                         </x>
                         <y>
-                        <noise type="gaussian">
-                            <mean>0.0</mean>
-                            <stddev>0.05236</stddev>
-                        </noise>
+                            <noise type="gaussian">
+                                <mean>0.0</mean>
+                                <stddev>0.00523598775</stddev>
+                                <bias_mean>0.0</bias_mean>
+                                <bias_stddev>0.05235987755</bias_stddev>
+                            </noise>
                         </y>
                         <z>
-                        <noise type="gaussian">
-                            <mean>0.0</mean>
-                            <stddev>0.05236</stddev>
-                        </noise>
+                            <noise type="gaussian">
+                                <mean>0.0</mean>
+                                <stddev>0.00523598775</stddev>
+                                <bias_mean>0.0</bias_mean>
+                                <bias_stddev>0.05235987755</bias_stddev>
+                            </noise>
                         </z>
                     </angular_velocity>
                     <linear_acceleration>
                         <x>
-                        <noise type="gaussian">
-                            <mean>0.0</mean>
-                            <stddev>1.8639e-5</stddev>
-                        </noise>
+                            <noise type="gaussian">
+                                <mean>0.0</mean>
+                                <stddev>1.8639e-5</stddev>
+                                <bias_mean>0.0</bias_mean>
+                                <bias_stddev>1.471e-3</bias_stddev>
+                            </noise>
                         </x>
                         <y>
@@ -43,4 +51,6 @@
                             <mean>0.0</mean>
                             <stddev>1.8639e-5</stddev>
+                            <bias_mean>0.0</bias_mean>
+                            <bias_stddev>1.471e-3</bias_stddev>
                         </noise>
                         </y>
@@ -49,4 +59,6 @@
                             <mean>0.0</mean>
                             <stddev>1.8639e-5</stddev>
+                            <bias_mean>0.0</bias_mean>
+                            <bias_stddev>1.471e-3</bias_stddev>
                         </noise>
                         </z>

File: vehicle_description/urdf/vehicle_core.urdf.xacro (robot description, xacro)
@@ -6,11 +6,11 @@
     <xacro:vehicle_wheels parent="vehicle_body"/>
     <xacro:imu_sensor name="imu1" topic_ns="imu1" parent="vehicle_body">
-        <origin xyz="0.05 0 ${(body_height / 2) + wheel_radius}" rpy="0 0 0"/>
+        <origin xyz="0 0 ${(body_height / 2) + wheel_radius}" rpy="0 0 0"/>
     </xacro:imu_sensor>
     <xacro:imu_sensor name="imu2" topic_ns="imu2" parent="vehicle_body">
-        <origin xyz="0 0 ${(body_height / 2) + wheel_radius}" rpy="0 0 0"></origin>
+        <origin xyz="0 0 ${(body_height / 2) + wheel_radius}" rpy="0 0 0"/>
     </xacro:imu_sensor>
     <xacro:imu_sensor name="imu3" topic_ns="imu3" parent="vehicle_body">
-        <origin xyz="-0.05 0 ${(body_height / 2) + wheel_radius}" rpy="0 0 0"></origin>
+        <origin xyz="0 0 ${(body_height / 2) + wheel_radius}" rpy="0 0 0"/>
     </xacro:imu_sensor>
 </robot>

Commit message: Imu ve Navsat modellerindeki parametere hataları giderildi

File: vehicle_description/urdf/includes/components/sensors/imu_gazebo.xacro (robot description, xacro)
@@ -83,7 +83,7 @@
                             <noise type="gaussian">
                                 <mean>0.0</mean>
-                                <stddev>9.94e-4</stddev>
+                                <stddev>6.11e-5</stddev> <!-- radyan cinsinden -->
                                 <bias_mean>0.0</bias_mean>
-                                <bias_stddev>4.848e-6</bias_stddev> <!-- radyan cinsinden -->
+                                <bias_stddev>4.848e-5</bias_stddev> <!-- radyan cinsinden -->
                             </noise>
                         </x>
@@ -91,15 +91,15 @@
                             <noise type="gaussian">
                                 <mean>0.0</mean>
-                                <stddev>9.94e-4</stddev>
+                                <stddev>6.11e-5</stddev>
                                 <bias_mean>0.0</bias_mean>
-                                <bias_stddev>4.848e-6</bias_stddev>
+                                <bias_stddev>4.848e-5</bias_stddev>
                             </noise>
                         </y>
                         <z>
-                            <noise type="gaussian">
+                             <noise type="gaussian">
                                 <mean>0.0</mean>
-                                <stddev>9.94e-4</stddev>
+                                <stddev>6.11e-5</stddev>
                                 <bias_mean>0.0</bias_mean>
-                                <bias_stddev>4.848e-6</bias_stddev>
+                                <bias_stddev>4.848e-5</bias_stddev>
                             </noise>
                         </z>
@@ -109,5 +109,5 @@
                             <noise type="gaussian">
                                 <mean>0.0</mean>
-                                <stddev>0.02082152953</stddev>
+                                <stddev>0.001373</stddev> <!-- m/s^2 cinsinden. -->
                                 <bias_mean>0.0</bias_mean>
                                 <bias_stddev>3.92e-4</bias_stddev> <!-- m/s^2 cinsinden. -->
@@ -117,5 +117,5 @@
                             <noise type="gaussian">
                                 <mean>0.0</mean>
-                                <stddev>0.02082152953</stddev>
+                                <stddev>0.001373</stddev>
                                 <bias_mean>0.0</bias_mean>
                                 <bias_stddev>3.92e-4</bias_stddev>
@@ -125,5 +125,5 @@
                             <noise type="gaussian">
                                 <mean>0.0</mean>
-                                <stddev>0.02082152953</stddev>
+                                <stddev>0.001373</stddev>
                                 <bias_mean>0.0</bias_mean>
                                 <bias_stddev>3.92e-4</bias_stddev>

File: vehicle_description/urdf/includes/components/sensors/navsat_gazebo.xacro (robot description, xacro)
@@ -1,5 +1,5 @@
 <?xml version="1.0" ?>
 <robot name="vehicle" xmlns:xacro="http://www.ros.org/wiki/xacro">
-    <!-- https://content.u-blox.com/sites/default/files/NEO-M8U_DataSheet_UBX-15015679.pdf -->
+    <!--https://www.vectornav.com/docs/default-source/product-brief/vn-200-product-brief.pdf?sfvrsn=5bda007a_2 -->
     <xacro:macro name="navsat_gazebo" params="navsat_name topic_ns">
         <gazebo reference="${navsat_name}">
@@ -10,10 +10,9 @@
                 <topic>${topic_ns}/fix</topic>
                 <navsat>
-                    <!-- Konum Ölçümü -->
                     <position_sensing>
                         <horizontal>
                             <noise type="gaussian">
                                 <mean>0.0</mean>
-                                <stddev>2.5</stddev> <!-- Yatay doğruluk (2.5 metre)  Not, SBAS ile 1.5 metre !! -->
+                                <stddev>1.0</stddev>
                             </noise>
                         </horizontal>
@@ -21,14 +20,13 @@
                             <noise type="gaussian">
                                 <mean>0.0</mean>
-                                <stddev>3.5</stddev> <!-- Dikey doğruluk (3.5 metre) (SBAS => uydu tabanlı arttırma sistemi) -->
+                                <stddev>1.5</stddev>
                             </noise>
                         </vertical>
                     </position_sensing>
-                    <!-- Hız Ölçümü -->
                     <velocity_sensing>
                         <horizontal>
                             <noise type="gaussian">
                                 <mean>0.0</mean>
-                                <stddev>0.05</stddev> <!-- Hız doğruluğu (0.05 m/s) -->
+                                <stddev>0.05</stddev>
                             </noise>
                         </horizontal>
@@ -36,16 +34,8 @@
                             <noise type="gaussian">
                                 <mean>0.0</mean>
-                                <stddev>0.1</stddev> <!-- Dikey hızda daha fazla hata -->
+                                <stddev>0.05</stddev>
                             </noise>
                         </vertical>
                     </velocity_sensing>
-                    <!-- ??
-                    <multipath>
-                        <noise type="gaussian">
-                            <mean>0.0</mean>
-                            <stddev>2.0</stddev>
-                        </noise>
-                    </multipath>
-                    -->
                 </navsat>
             </sensor>

File: vehicle_description/urdf/includes/components/sensors/navsat_sensor.xacro (robot description, xacro)
@@ -2,27 +2,11 @@
 <robot name="vehicle" xmlns:xacro="http://www.ros.org/wiki/xacro">
     <xacro:include filename="$(find vehicle_description)/urdf/includes/components/sensors/navsat_gazebo.xacro" />
-    <xacro:macro name="navsat_sensor" params="name topic_ns:=navsat parent *origin">
-        <joint name="${name}_joint" type="fixed">
-            <parent link="${parent}"/>
-            <child link="${name}"/>
-            <xacro:insert_block name="origin" />
-        </joint>
-        <link name="${name}">
-            <visual>
-                <origin xyz="0 0 0"/>
-                <geometry>
-                    <box size="0.01 0.01 0.01"/>
-                </geometry>
-                <material name="silver"/>
-            </visual>
-            <collision>
-                <origin xyz="0 0 0"/>
-                <geometry>
-                    <box size="0.01 0.01 0.01"/>
-                </geometry>
-            </collision>
-            <xacro:solid_cuboid_inertia mass="0.01" x="0.01" y="0.01" z="0.01" />
-        </link>
-        <xacro:navsat_gazebo navsat_name="${name}" topic_ns="${topic_ns}"/>
+    <xacro:include filename="$(find vehicle_description)/urdf/includes/components/sensors/vn200.xacro" />
+    <xacro:macro name="navsat_sensor" params="sensor_type name topic_ns:=imu parent *origin">
+        <xacro:if value="${sensor_type == 'vn_200'}">
+            <xacro:vn_100 name="${name}" topic_ns="${topic_ns}" parent="${parent}">
+                <xacro:insert_block name="origin"/>
+            </xacro:vn_100>
+        </xacro:if>
     </xacro:macro>
 </robot>

File: vehicle_description/urdf/includes/components/sensors/vn100.xacro (robot description, xacro)
@@ -3,6 +3,6 @@
     <xacro:include filename="$(find vehicle_description)/urdf/includes/components/sensors/imu_gazebo.xacro" />
     <!-- VN100 CONSTANST https://www.vectornav.com/docs/default-source/product-brief/vn-100-product-brief.pdf?sfvrsn=a2a5ae5f_2 -->
+    <xacro:property name="vn100_width" value="0.024" />
     <xacro:property name="vn100_depth" value="0.022" />
-    <xacro:property name="vn100_width" value="0.024" />
     <xacro:property name="vn100_height" value="0.003"/>
     <xacro:property name="vn100_mass" value="0.0035"/>

File: vehicle_description/urdf/vehicle_core.urdf.xacro (robot description, xacro)
@@ -14,5 +14,5 @@
         <origin xyz="0 0 ${(body_height / 2) + 0.0015 + wheel_radius}" rpy="0 0 0"/>
     </xacro:imu_sensor>
-    <xacro:navsat_sensor name="gps" topic_ns="navsat" parent="base_link" >
+    <xacro:navsat_sensor sensor_type="vn_200" name="gps" topic_ns="navsat" parent="base_link" >
         <origin xyz="0.1 0 ${(body_height / 2) + 0.005 + wheel_radius}" rpy="0 0 0" />
     </xacro:navsat_sensor>
