Commit message: Imu logger artık hem csv hem de xlsx çıktısı uretiyor

File: vehicle_description/urdf/includes/components/body/vehicle_body.xacro (robot description, xacro)
@@ -2,13 +2,13 @@
 <robot name="vehicle" xmlns:xacro="http://www.ros.org/wiki/xacro">
     <!-- Vehicle Body Parameters -->
-    <xacro:property name="body_width"  value="0.6" />
-    <xacro:property name="body_depth"  value="0.5" />
-    <xacro:property name="body_height" value="0.2" />
-    <xacro:property name="body_mass" value="2" />
+    <xacro:property name="body_width"  value="0.3" />
+    <xacro:property name="body_depth"  value="0.25" />
+    <xacro:property name="body_height" value="0.1" />
+    <xacro:property name="body_mass" value="3" />
     <!-- WHEEL PROPERTIES-->
-    <xacro:property name="wheel_radius" value="0.1"/>
+    <xacro:property name="wheel_radius" value="0.05"/>
     <xacro:property name="wheel_length" value="0.05" />
     <xacro:property name="wheel_mass" value="0.5" />
-    <xacro:property name="caster_wheel_radius" value="0.1" />
+    <xacro:property name="caster_wheel_radius" value="0.05" />
     <xacro:property name="caster_wheel_mass" value="0.5"/>
     <xacro:macro name="vehicle_body">

File: vehicle_description/urdf/includes/components/sensors/imu_gazebo.xacro (robot description, xacro)
@@ -26,5 +26,5 @@
                                 <stddev>0.00523598775</stddev>
                                 <bias_mean>0.0</bias_mean>
-                                <bias_stddev>0.05235987755</bias_stddev>
+                                <bias_stddev>0.0005235987755</bias_stddev>
                             </noise>
                         </y>

File: vehicle_description/urdf/includes/components/wheels/vehicle_wheels.xacro (robot description, xacro)
@@ -1,15 +1,4 @@
 <?xml version="1.0"?>
 <robot name="vehicle" xmlns:xacro="http://www.ros.org/wiki/xacro">
-    <!-- Vehicle Body Parameters -->
-    <xacro:property name="body_width"  value="0.6" />
-    <xacro:property name="body_depth"  value="0.5" />
-    <xacro:property name="body_height" value="0.2" />
-    <xacro:property name="body_mass" value="2" />
-    <!-- WHEEL PROPERTIES-->
-    <xacro:property name="wheel_radius" value="0.1"/>
-    <xacro:property name="wheel_length" value="0.05" />
-    <xacro:property name="wheel_mass" value="0.5" />
-    <xacro:property name="caster_wheel_radius" value="0.1" />
-    <xacro:property name="caster_wheel_mass" value="0.5"/>
     <xacro:macro name="vehicle_wheels" params="parent">
         <link name="rear_right_wheel">

Commit message: Hata var!

File: vehicle_description/urdf/includes/components/body/vehicle_body.xacro (robot description, xacro)
@@ -5,17 +5,19 @@
     <xacro:property name="body_depth"  value="0.25" />
     <xacro:property name="body_height" value="0.1" />
-    <xacro:property name="body_mass" value="3" />
+    <xacro:property name="body_mass" value="5" />
     <!-- WHEEL PROPERTIES-->
     <xacro:property name="wheel_radius" value="0.05"/>
     <xacro:property name="wheel_length" value="0.05" />
+    <xacro:property name="wheel_zoff" value="0.07"/>
     <xacro:property name="wheel_mass" value="0.5" />
     <xacro:property name="caster_wheel_radius" value="0.05" />
     <xacro:property name="caster_wheel_mass" value="0.5"/>
     <xacro:macro name="vehicle_body">
-        <link name="base_footprint" />
+        <link name="base_footprint" >
+            <xacro:solid_cuboid_inertia mass="0" x="0" y="0" z="0"/>
+        </link>
         <!-- Base Link -->
-        <link name="vehicle_body">
+        <link name="base_link">
             <visual>
-                <origin xyz ="0 0 ${wheel_radius}" />
                 <geometry>
                     <box size="${body_width} ${body_depth} ${body_height}"/>
@@ -24,5 +26,4 @@
             </visual>
             <collision>
-                <origin xyz ="0 0 ${wheel_radius}" />
                 <geometry>
                     <box size="${body_width} ${body_depth} ${body_height}"/>
@@ -31,8 +32,8 @@
             <xacro:solid_cuboid_inertia mass="${body_mass}" x="${body_width}" y="${body_depth}" z="${body_height}" />
         </link>
-        <joint name="vehicle_body_joint" type="fixed">
-            <parent link="base_footprint"/>
-            <child link="vehicle_body" />
-            <origin xyz="0 0 ${body_height / 2}"/>
+        <joint name="base_link_joint" type="fixed">
+            <parent link="base_link"/>
+            <child link="base_footprint" />
+            <origin xyz="0 0 ${-(wheel_radius)}"/>
         </joint>
     </xacro:macro>

File: vehicle_description/urdf/includes/components/sensors/imu_gazebo.xacro (robot description, xacro)
@@ -76,5 +76,5 @@
                 <always_on>true</always_on>
                 <update_rate>200</update_rate>
-                <gz_fram_id>${imu_name}_link</gz_fram_id>
+                <gz_frame_id>${imu_name}_link</gz_frame_id>
                 <topic>${topic_ns}</topic>
                 <imu>

File: vehicle_description/urdf/includes/components/sensors/navsat_gazebo.xacro (robot description, xacro)
@@ -2,10 +2,10 @@
 <robot name="vehicle" xmlns:xacro="http://www.ros.org/wiki/xacro">
     <xacro:macro name="navsat_gazebo" params="navsat_name topic_ns">
-        <gazebo reference="${navsat_name}_link">
+        <gazebo reference="${navsat_name}">
             <sensor name="${navsat_name}" type="navsat">
                 <always_on>1</always_on>
-                <update_rate>10</update_rate>
-                <pose>0 0 0 0 0 0</pose>
-                <topic>${topic_ns}</topic>
+                <pose>0 0 0.05 0 0 0</pose>
+                <update_rate>50</update_rate>
+                <topic>${topic_ns}/fix</topic>
                 <navsat>
                     <position_sensing>
@@ -13,5 +13,5 @@
                             <noise type="gaussian">
                                 <mean>0.0</mean>
-                                <stddev>0.002</stddev>
+                                <stddev>0.0</stddev>
                             </noise>
                         </horizontal>
@@ -19,5 +19,5 @@
                             <noise type="gaussian">
                                 <mean>0.0</mean>
-                                <stddev>0.002</stddev>
+                                <stddev>0.0</stddev>
                             </noise>
                         </vertical>
@@ -27,5 +27,5 @@
                             <noise type="gaussian">
                                 <mean>0.0</mean>
-                                <stddev>0.002</stddev>
+                                <stddev>0.0</stddev>
                             </noise>
                         </horizontal>
@@ -33,5 +33,5 @@
                             <noise type="gaussian">
                                 <mean>0.0</mean>
-                                <stddev>0.002</stddev>
+                                <stddev>0.0</stddev>
                             </noise>
                         </vertical>

File: vehicle_description/urdf/includes/components/sensors/navsat_sensor.xacro (robot description, xacro)
@@ -2,15 +2,15 @@
 <robot name="vehicle" xmlns:xacro="http://www.ros.org/wiki/xacro">
     <xacro:include filename="$(find vehicle_description)/urdf/includes/components/sensors/navsat_gazebo.xacro" />
-    <xacro:macro name="navsat_sensor" params="name topic_ns:=imu parent *origin">
+    <xacro:macro name="navsat_sensor" params="name topic_ns:=navsat parent *origin">
         <joint name="${name}_joint" type="fixed">
             <parent link="${parent}"/>
-            <child link="${name}_link"/>
+            <child link="${name}"/>
             <xacro:insert_block name="origin" />
         </joint>
-        <link name="${name}_link">
+        <link name="${name}">
             <visual>
                 <origin xyz="0 0 0"/>
                 <geometry>
-                    <box size="0.001 0.001 0.001"/>
+                    <box size="0.01 0.01 0.01"/>
                 </geometry>
                 <material name="silver"/>
@@ -19,8 +19,8 @@
                 <origin xyz="0 0 0"/>
                 <geometry>
-                    <box size="0.001 0.001 0.001"/>
+                    <box size="0.01 0.01 0.01"/>
                 </geometry>
             </collision>
-            <xacro:solid_cuboid_inertia mass="0.001" x="0.001" y="0.001" z="0.001" />
+            <xacro:solid_cuboid_inertia mass="0.01" x="0.01" y="0.01" z="0.01" />
         </link>
         <xacro:navsat_gazebo navsat_name="${name}" topic_ns="${topic_ns}"/>

File: vehicle_description/urdf/includes/gazebo/gazebo_system.xacro (robot description, xacro)
@@ -42,5 +42,7 @@
         <plugin filename="ignition-gazebo-odometry-publisher-system" name="ignition::gazebo::systems::OdometryPublisher">
             <odom_frame>odom</odom_frame>
-            <robot_base_frame>vehicle_body</robot_base_frame>
+            <odom_covariance_topic>odom</odom_covariance_topic>
+            <tf_topic>tf</tf_topic>
+            <robot_base_frame>base_link</robot_base_frame>
             <update_rate>100</update_rate>
             <publish_odom_tf>true</publish_odom_tf>

File: vehicle_description/urdf/vehicle_core.urdf.xacro (robot description, xacro)
@@ -4,16 +4,16 @@
     <xacro:include filename="$(find vehicle_description)/urdf/includes.xacro" />
     <xacro:vehicle_body />
-    <xacro:vehicle_wheels parent="vehicle_body"/>
-    <xacro:imu_sensor sensor_type="vn_100" name="imu1" topic_ns="imu1" parent="vehicle_body">
+    <xacro:vehicle_wheels parent="base_link"/>
+    <xacro:imu_sensor sensor_type="vn_100" name="imu1" topic_ns="imu1" parent="base_link">
         <origin xyz="0 0 ${(body_height / 2) + wheel_radius}" rpy="0 0 0"/>
     </xacro:imu_sensor>
-    <xacro:imu_sensor sensor_type="vn_100" name="imu2" topic_ns="imu2" parent="vehicle_body">
+    <xacro:imu_sensor sensor_type="vn_100" name="imu2" topic_ns="imu2" parent="base_link">
         <origin xyz="0 0 ${(body_height / 2) + wheel_radius}" rpy="0 0 0"/>
     </xacro:imu_sensor>
-    <xacro:imu_sensor sensor_type="vn_100" name="imu3" topic_ns="imu3" parent="vehicle_body">
+    <xacro:imu_sensor sensor_type="vn_100" name="imu3" topic_ns="imu3" parent="base_link">
         <origin xyz="0 0 ${(body_height / 2) + wheel_radius}" rpy="0 0 0"/>
     </xacro:imu_sensor>
-    <xacro:navsat_sensor name="gps" topic_ns="navsat" parent="vehicle_body" >
-        <origin xyz="0.05 0 ${(body_height / 2) + wheel_radius}" rpy="0 0 0" />
+    <xacro:navsat_sensor name="gps" topic_ns="navsat" parent="base_link" >
+        <origin xyz="0.1 0 ${(body_height / 2) + wheel_radius + 0.005}" rpy="0 0 0" />
     </xacro:navsat_sensor>
 </robot>

Commit message: Hatalar düzeltildi

File: vehicle_description/urdf/includes/components/body/vehicle_body.xacro (robot description, xacro)
@@ -5,19 +5,18 @@
     <xacro:property name="body_depth"  value="0.25" />
     <xacro:property name="body_height" value="0.1" />
-    <xacro:property name="body_mass" value="5" />
+    <xacro:property name="body_mass" value="3" />
     <!-- WHEEL PROPERTIES-->
     <xacro:property name="wheel_radius" value="0.05"/>
     <xacro:property name="wheel_length" value="0.05" />
-    <xacro:property name="wheel_zoff" value="0.07"/>
+    <xacro:property name="wheel_zoff" value="0.025"/>
     <xacro:property name="wheel_mass" value="0.5" />
     <xacro:property name="caster_wheel_radius" value="0.05" />
     <xacro:property name="caster_wheel_mass" value="0.5"/>
     <xacro:macro name="vehicle_body">
-        <link name="base_footprint" >
-            <xacro:solid_cuboid_inertia mass="0" x="0" y="0" z="0"/>
-        </link>
+        <link name="base_footprint" />
         <!-- Base Link -->
         <link name="base_link">
             <visual>
+                <origin xyz="0 0 0"/>
                 <geometry>
                     <box size="${body_width} ${body_depth} ${body_height}"/>
@@ -26,4 +25,5 @@
             </visual>
             <collision>
+                <origin xyz="0 0 0"/>
                 <geometry>
                     <box size="${body_width} ${body_depth} ${body_height}"/>
@@ -33,7 +33,7 @@
         </link>
         <joint name="base_link_joint" type="fixed">
-            <parent link="base_link"/>
-            <child link="base_footprint" />
-            <origin xyz="0 0 ${-(wheel_radius)}"/>
+            <parent link="base_footprint"/>
+            <child link="base_link" />
+            <origin xyz="0 0 ${(wheel_radius + wheel_zoff)}" rpy="0 0 0"/>
         </joint>
     </xacro:macro>

File: vehicle_description/urdf/includes/components/wheels/vehicle_wheels.xacro (robot description, xacro)
@@ -53,5 +53,5 @@
             <parent link="${parent}"/>
             <child link="rear_right_wheel"/>
-            <origin xyz="${-(body_width / 4)} ${((body_depth / 2) + (wheel_length / 2))} 0" rpy="-${pi/2} 0 0"/>
+            <origin xyz="${-(body_width / 4)} ${((body_depth / 2) + (wheel_length / 2))} ${-wheel_zoff}" rpy="-${pi/2} 0 0"/>
             <axis xyz="0 0 1"/>
             <!-- <dynamics damping="0.2" /> -->
@@ -60,5 +60,5 @@
             <parent link="${parent}"/>
             <child link="rear_left_wheel"/>
-            <origin xyz="${-(body_width / 4)} ${-((body_depth / 2) + (wheel_length / 2))} 0" rpy="-${pi/2} 0 0"/>
+            <origin xyz="${-(body_width / 4)} ${-((body_depth / 2) + (wheel_length / 2))} ${-wheel_zoff}" rpy="-${pi/2} 0 0"/>
             <axis xyz="0 0 1"/>
             <!-- <dynamics damping="0.2" /> -->
@@ -67,5 +67,5 @@
             <parent link="${parent}"/>
             <child  link="front_caster_wheel"/>
-            <origin xyz="${body_width / 4} 0 0"/>
+            <origin xyz="${body_width / 4} 0 ${-wheel_zoff}"/>
         </joint>
     </xacro:macro>

File: vehicle_description/urdf/includes/gazebo/gazebo_system.xacro (robot description, xacro)
@@ -42,8 +42,6 @@
         <plugin filename="ignition-gazebo-odometry-publisher-system" name="ignition::gazebo::systems::OdometryPublisher">
             <odom_frame>odom</odom_frame>
-            <odom_covariance_topic>odom</odom_covariance_topic>
-            <tf_topic>tf</tf_topic>
             <robot_base_frame>base_link</robot_base_frame>
-            <update_rate>100</update_rate>
+            <odom_publish_frequency>200</odom_publish_frequency>
             <publish_odom_tf>true</publish_odom_tf>
             <dimensions>3</dimensions>

Commit message: Ros2 control kısmı çözülemedi ama hatalar giderildi

File: vehicle_description/urdf/includes/components/body/vehicle_body.xacro (robot description, xacro)
@@ -5,9 +5,8 @@
     <xacro:property name="body_depth"  value="0.25" />
     <xacro:property name="body_height" value="0.1" />
-    <xacro:property name="body_mass" value="3" />
+    <xacro:property name="body_mass" value="2" />
     <!-- WHEEL PROPERTIES-->
     <xacro:property name="wheel_radius" value="0.05"/>
     <xacro:property name="wheel_length" value="0.05" />
-    <xacro:property name="wheel_zoff" value="0.025"/>
     <xacro:property name="wheel_mass" value="0.5" />
     <xacro:property name="caster_wheel_radius" value="0.05" />
@@ -18,5 +17,5 @@
         <link name="base_link">
             <visual>
-                <origin xyz="0 0 0"/>
+                <origin xyz="0 0 ${wheel_radius}"/>
                 <geometry>
                     <box size="${body_width} ${body_depth} ${body_height}"/>
@@ -25,5 +24,5 @@
             </visual>
             <collision>
-                <origin xyz="0 0 0"/>
+                <origin xyz="0 0 ${wheel_radius}"/>
                 <geometry>
                     <box size="${body_width} ${body_depth} ${body_height}"/>
@@ -35,5 +34,5 @@
             <parent link="base_footprint"/>
             <child link="base_link" />
-            <origin xyz="0 0 ${(wheel_radius + wheel_zoff)}" rpy="0 0 0"/>
+            <origin xyz="0 0 ${(body_height / 2)}" rpy="0 0 0"/>
         </joint>
     </xacro:macro>

File: vehicle_description/urdf/includes/components/sensors/navsat_gazebo.xacro (robot description, xacro)
@@ -15,5 +15,5 @@
                             <noise type="gaussian">
                                 <mean>0.0</mean>
-                                <stddev>2.5</stddev> <!-- Yatay doğruluk (2.5 metre)  Not: SBAS ile 1.5 metre !! -->
+                                <stddev>2.5</stddev> <!-- Yatay doğruluk (2.5 metre)  Not, SBAS ile 1.5 metre !! -->
                             </noise>
                         </horizontal>
@@ -21,5 +21,5 @@
                             <noise type="gaussian">
                                 <mean>0.0</mean>
-                                <stddev>3.5</stddev> <!-- Dikey doğruluk (3.5 metre) (SBAS => uydu tabanlı arttırma sistemi)-->
+                                <stddev>3.5</stddev> <!-- Dikey doğruluk (3.5 metre) (SBAS => uydu tabanlı arttırma sistemi) -->
                             </noise>
                         </vertical>

File: vehicle_description/urdf/includes/components/wheels/vehicle_wheels.xacro (robot description, xacro)
@@ -50,9 +50,10 @@
             <xacro:sphere_inertia mass="${caster_wheel_mass}" r="${caster_wheel_radius}" />
         </link>
+W
         <joint name="rear_right_wheel_joint" type="continuous">
             <parent link="${parent}"/>
             <child link="rear_right_wheel"/>
-            <origin xyz="${-(body_width / 4)} ${-((body_depth / 2) + (wheel_length / 2))} ${-wheel_zoff}" rpy="-${pi/2} 0 0"/>
-            <axis xyz="0 0 1"/>
+            <origin xyz="${-(body_width / 4)} ${-((body_depth / 2) + (wheel_length / 2))} 0" rpy="${pi/2} 0 0"/>
+            <axis xyz="0 0 -1"/>
             <!-- <dynamics damping="0.2" /> -->
         </joint>
@@ -60,5 +61,5 @@
             <parent link="${parent}"/>
             <child link="rear_left_wheel"/>
-            <origin xyz="${-(body_width / 4)} ${((body_depth / 2) + (wheel_length / 2))} ${-wheel_zoff}" rpy="-${pi/2} 0 0"/>
+            <origin xyz="${-(body_width / 4)} ${((body_depth / 2) + (wheel_length / 2))} 0" rpy="-${pi/2} 0 0"/>
             <axis xyz="0 0 1"/>
             <!-- <dynamics damping="0.2" /> -->
@@ -67,5 +68,5 @@
             <parent link="${parent}"/>
             <child  link="front_caster_wheel"/>
-            <origin xyz="${body_width / 4} 0 ${-wheel_zoff}"/>
+            <origin xyz="${body_width / 4} 0 0"/>
         </joint>
     </xacro:macro>

File: vehicle_description/urdf/includes/gazebo/gazebo_system.xacro (robot description, xacro)
@@ -2,20 +2,20 @@
 <robot name="vehicle" xmlns="http://www.ros.org/wiki/xacro">
     <gazebo references="rear_right_wheel">
-        <mu1>10000</mu1>
-        <mu2>10000</mu2>
-        <kp>10000</kp>
+        <mu1>1000000000000000.0</mu1>
+        <mu2>1000000000000000.0</mu2>
+        <kp>1000000000000.0</kp>
         <kd>10.0</kd>
         <minDepth>0.001</minDepth>
         <maxVel>0.1</maxVel>
-        <fdirl>1 0 0</fdirl>
+        <fdirl>0 0 1</fdirl>
     </gazebo>
     <gazebo references="rear_left_wheel">
-        <mu1>10000</mu1>
-        <mu2>10000</mu2>
-        <kp>10000</kp>
+        <mu1>1000000000000000.0</mu1>
+        <mu2>1000000000000000.0</mu2>
+        <kp>1000000000000000.0</kp>
         <kd>10.0</kd>
         <minDepth>0.001</minDepth>
         <maxVel>0.1</maxVel>
-        <fdirl>1 0 0</fdirl>
+        <fdirl>0 0 1</fdirl>
     </gazebo>
     <gazebo references="front_caster_wheel">
@@ -25,6 +25,5 @@
         <kd>100.0</kd>
         <minDepth>0.001</minDepth>
-        <maxVel>0.1</maxVel>
-        <fdirl>1 0 0</fdirl>
+        <maxVel>1.0</maxVel>
     </gazebo>
     <!-- ?? -->
@@ -49,5 +48,5 @@
     </gazebo>
     <!-- Donanım ile etkileşime geçen kısmı ayarladığımız nokta !! -->
-    <ros2_control name="IgnitionSystem" type="system" >
+    <ros2_control name="RobotSystem" type="system" >
         <!-- use mock hardware gerçek bir robota yükleme yaparken kullanılır! -->
         <hardware>
@@ -56,6 +55,6 @@
         <joint name="rear_right_wheel_joint">
             <command_interface name="velocity">
-                <param name="min">-5</param>
-                <param name="max">5</param>
+                <param name="min">-1</param>
+                <param name="max">1</param>
             </command_interface>
             <state_interface name="position" />
@@ -64,6 +63,6 @@
         <joint name="rear_left_wheel_joint">
             <command_interface name="velocity">
-                <param name="min">-5</param>
-                <param name="max">5</param>
+                <param name="min">-1</param>
+                <param name="max">1</param>
             </command_interface>
             <state_interface name="position" />

File: vehicle_description/urdf/includes/gazebo/inertias.xacro (robot description, xacro)
@@ -5,4 +5,7 @@
     <xacro:macro name="solid_cuboid_inertia" params="mass x y z">
         <inertial>
+            <!--
+            <xacro:insert_block name="origin"/>
+            -->
             <mass value="${mass}"/>
             <inertia ixx="${mass * (y * y + z * z) / 12}" ixy="0" ixz="0"
@@ -14,4 +17,7 @@
     <xacro:macro name="cylinder_inertia" params="mass r h">
         <inertial>
+            <!--
+            <xacro:insert_block name="origin"/>
+            -->
             <mass value="${mass}" />
             <inertia ixx="${mass * (3 * r * r + h * h) / 12}" ixy="0" ixz="0"
@@ -23,4 +29,7 @@
     <xacro:macro name="sphere_inertia" params="mass r">
         <inertial>
+            <!--
+            <xacro:insert_block name="origin"/>
+            -->
             <mass value="${mass}" />
             <inertia ixx="${mass * (2 * r * r) / 5}" ixy="0" ixz="0"

File: vehicle_description/urdf/vehicle_core.urdf.xacro (robot description, xacro)
@@ -6,14 +6,14 @@
     <xacro:vehicle_wheels parent="base_link"/>
     <xacro:imu_sensor sensor_type="vn_100" name="imu1" topic_ns="imu1" parent="base_link">
-        <origin xyz="0 0 ${(body_height / 2)}" rpy="0 0 0"/>
+        <origin xyz="0 0 ${(body_height / 2) + 0.0015 + wheel_radius}" rpy="0 0 0"/>
     </xacro:imu_sensor>
     <xacro:imu_sensor sensor_type="vn_100" name="imu2" topic_ns="imu2" parent="base_link">
-        <origin xyz="0 0 ${(body_height / 2)}" rpy="0 0 0"/>
+        <origin xyz="0 0 ${(body_height / 2) + 0.0015 + wheel_radius}" rpy="0 0 0"/>
     </xacro:imu_sensor>
     <xacro:imu_sensor sensor_type="vn_100" name="imu3" topic_ns="imu3" parent="base_link">
-        <origin xyz="0 0 ${(body_height / 2)}" rpy="0 0 0"/>
+        <origin xyz="0 0 ${(body_height / 2) + 0.0015 + wheel_radius}" rpy="0 0 0"/>
     </xacro:imu_sensor>
     <xacro:navsat_sensor name="gps" topic_ns="navsat" parent="base_link" >
-        <origin xyz="0.1 0 ${(body_height / 2) + 0.005}" rpy="0 0 0" />
+        <origin xyz="0.1 0 ${(body_height / 2) + 0.005 + wheel_radius}" rpy="0 0 0" />
     </xacro:navsat_sensor>
 </robot>
