Commit message: refactoring gazebo launch file

File: vehicle_description/urdf/includes/components/wheels/vehicle_wheels.xacro (robot description, xacro)
@@ -53,5 +53,5 @@
             <parent link="${parent}"/>
             <child link="rear_right_wheel"/>
-            <origin xyz="${-(body_width / 4)} ${((body_depth / 2) + (wheel_length / 2))} ${-wheel_zoff}" rpy="-${pi/2} 0 0"/>
+            <origin xyz="${-(body_width / 4)} ${-((body_depth / 2) + (wheel_length / 2))} ${-wheel_zoff}" rpy="-${pi/2} 0 0"/>
             <axis xyz="0 0 1"/>
             <!-- <dynamics damping="0.2" /> -->
@@ -60,5 +60,5 @@
             <parent link="${parent}"/>
             <child link="rear_left_wheel"/>
-            <origin xyz="${-(body_width / 4)} ${-((body_depth / 2) + (wheel_length / 2))} ${-wheel_zoff}" rpy="-${pi/2} 0 0"/>
+            <origin xyz="${-(body_width / 4)} ${((body_depth / 2) + (wheel_length / 2))} ${-wheel_zoff}" rpy="-${pi/2} 0 0"/>
             <axis xyz="0 0 1"/>
             <!-- <dynamics damping="0.2" /> -->

File: vehicle_description/urdf/includes/gazebo/gazebo_system.xacro (robot description, xacro)
@@ -56,6 +56,6 @@
         <joint name="rear_right_wheel_joint">
             <command_interface name="velocity">
-                <param name="min">-1</param>
-                <param name="max">1</param>
+                <param name="min">-5</param>
+                <param name="max">5</param>
             </command_interface>
             <state_interface name="position" />
@@ -64,6 +64,6 @@
         <joint name="rear_left_wheel_joint">
             <command_interface name="velocity">
-                <param name="min">-1</param>
-                <param name="max">1</param>
+                <param name="min">-5</param>
+                <param name="max">5</param>
             </command_interface>
             <state_interface name="position" />

File: vehicle_description/urdf/vehicle_core.urdf.xacro (robot description, xacro)
@@ -6,14 +6,14 @@
     <xacro:vehicle_wheels parent="base_link"/>
     <xacro:imu_sensor sensor_type="vn_100" name="imu1" topic_ns="imu1" parent="base_link">
-        <origin xyz="0 0 ${(body_height / 2) + wheel_radius}" rpy="0 0 0"/>
+        <origin xyz="0 0 ${(body_height / 2)}" rpy="0 0 0"/>
     </xacro:imu_sensor>
     <xacro:imu_sensor sensor_type="vn_100" name="imu2" topic_ns="imu2" parent="base_link">
-        <origin xyz="0 0 ${(body_height / 2) + wheel_radius}" rpy="0 0 0"/>
+        <origin xyz="0 0 ${(body_height / 2)}" rpy="0 0 0"/>
     </xacro:imu_sensor>
     <xacro:imu_sensor sensor_type="vn_100" name="imu3" topic_ns="imu3" parent="base_link">
-        <origin xyz="0 0 ${(body_height / 2) + wheel_radius}" rpy="0 0 0"/>
+        <origin xyz="0 0 ${(body_height / 2)}" rpy="0 0 0"/>
     </xacro:imu_sensor>
     <xacro:navsat_sensor name="gps" topic_ns="navsat" parent="base_link" >
-        <origin xyz="0.1 0 ${(body_height / 2) + wheel_radius + 0.005}" rpy="0 0 0" />
+        <origin xyz="0.1 0 ${(body_height / 2) + 0.005}" rpy="0 0 0" />
     </xacro:navsat_sensor>
 </robot>

Commit message: Sensor fusion kısmı tamamlandı

File: vehicle_description/urdf/includes/components/wheels/vehicle_wheels.xacro (robot description, xacro)
@@ -56,5 +56,5 @@
             <origin xyz="${-(body_width / 4)} ${-((body_depth / 2) + (wheel_length / 2))} 0" rpy="${pi/2} 0 0"/>
             <axis xyz="0 0 -1"/>
-            <!-- <dynamics damping="0.2" /> -->
+            <!-- <dynamics damping="0.1" /> -->
         </joint>
         <joint name="rear_left_wheel_joint" type="continuous">
@@ -63,5 +63,5 @@
             <origin xyz="${-(body_width / 4)} ${((body_depth / 2) + (wheel_length / 2))} 0" rpy="-${pi/2} 0 0"/>
             <axis xyz="0 0 1"/>
-            <!-- <dynamics damping="0.2" /> -->
+            <!-- <dynamics damping="0.1" /> -->
         </joint>
         <joint name="front_caster_wheel_joint" type="fixed">

File: vehicle_description/urdf/includes/gazebo/gazebo_system.xacro (robot description, xacro)
@@ -22,5 +22,5 @@
         <mu1>0.1</mu1>
         <mu2>0.1</mu2>
-        <kp>1000000.0</kp>
+        <kp>1000000000.0</kp>
         <kd>100.0</kd>
         <minDepth>0.001</minDepth>
